Commit message: Shrank joint limits to make planner look smarter.

File: motoman_mh5_support/urdf/mh5_macro.xacro (robot description, xacro)
@@ -124,5 +124,5 @@
 			<origin xyz="0 0 0.1990" rpy="0 0 0"/>
 			<axis xyz="0 0 1" />
-			<limit lower="-2.9671" upper="2.9671" effort="100" velocity="2.96" />
+			<limit lower="-2.9671" upper="1.571" effort="100" velocity="2.96" />
 		</joint>
 		<joint name="${prefix}joint_l" type="revolute">
@@ -138,5 +138,5 @@
 			<origin xyz="0 0 0.3100" rpy="0 0 0"/>
 			<axis xyz="0 -1 0" />
-			<limit lower="-2.3736" upper="4.4506" effort="100" velocity="2.96" />
+			<limit lower="-2.3736" upper="1.571" effort="100" velocity="2.96" />
 		</joint>
 		<joint name="${prefix}joint_r" type="revolute">
@@ -145,5 +145,5 @@
 			<origin xyz="0.0715 0 0.0399" rpy="0 0 0"/>
 			<axis xyz="-1 0 0" />
-			<limit lower="-3.3161" upper="3.3161" effort="100" velocity="3.48" />
+			<limit lower="-1.571" upper="1.571" effort="100" velocity="3.48" />
 		</joint>
 		<joint name="${prefix}joint_b" type="revolute">
@@ -159,5 +159,5 @@
 			<origin xyz="0.0510 0 0" rpy="0 0 0"/>
 			<axis xyz="-1 0 0" />
-			<limit lower="-6.2831" upper="6.2831" effort="100" velocity="6.97" />
+			<limit lower="-3.15" upper="3.15" effort="100" velocity="6.97" />
 		</joint>
 		<!-- end of joint list -->

Commit message: Increased speed limits to match spec sheet.

File: motoman_mh5_support/urdf/mh5_macro.xacro (robot description, xacro)
@@ -124,5 +124,5 @@
 			<origin xyz="0 0 0.1990" rpy="0 0 0"/>
 			<axis xyz="0 0 1" />
-			<limit lower="-2.9671" upper="2.9671" effort="100" velocity="2.96" />
+			<limit lower="-2.9671" upper="2.9671" effort="100" velocity="6.56" />
 		</joint>
 		<joint name="${prefix}joint_l" type="revolute">
@@ -131,5 +131,5 @@
 			<origin xyz="0.0880 0 0.1310" rpy="0 0 0"/>
 			<axis xyz="0 1 0" />
-			<limit lower="-1.1345" upper="2.6180" effort="100" velocity="2.96" />
+			<limit lower="-1.1345" upper="2.6180" effort="100" velocity="6.1" />
 		</joint>
 		<joint name="${prefix}joint_u" type="revolute">
@@ -138,5 +138,5 @@
 			<origin xyz="0 0 0.3100" rpy="0 0 0"/>
 			<axis xyz="0 -1 0" />
-			<limit lower="-2.3736" upper="4.4506" effort="100" velocity="2.96" />
+			<limit lower="-2.3736" upper="4.4506" effort="100" velocity="6.98" />
 		</joint>
 		<joint name="${prefix}joint_r" type="revolute">
@@ -145,5 +145,5 @@
 			<origin xyz="0.0715 0 0.0399" rpy="0 0 0"/>
 			<axis xyz="-1 0 0" />
-			<limit lower="-3.3161" upper="3.3161" effort="100" velocity="3.48" />
+			<limit lower="-3.3161" upper="3.3161" effort="100" velocity="7.85" />
 		</joint>
 		<joint name="${prefix}joint_b" type="revolute">
@@ -152,5 +152,5 @@
 			<origin xyz="0.2335 0 0" rpy="0 0 0"/>
 			<axis xyz="0 -1 0" />
-			<limit lower="-2.1817" upper="2.1817" effort="100" velocity="3.48" />
+			<limit lower="-2.1817" upper="2.1817" effort="100" velocity="7.85" />
 		</joint>
 		<joint name="${prefix}joint_t" type="revolute">
@@ -159,5 +159,5 @@
 			<origin xyz="0.0510 0 0" rpy="0 0 0"/>
 			<axis xyz="-1 0 0" />
-			<limit lower="-6.2831" upper="6.2831" effort="100" velocity="6.97" />
+			<limit lower="-6.2831" upper="6.2831" effort="100" velocity="12.56" />
 		</joint>
 		<!-- end of joint list -->
